File: _autosave-CAN_Shield.kicad_sch (KiCad schematic)
At the start: 17 parts, among them J1 GPIO, U1 MX128-5.08-09P-GN01-CU-Y-A, U2 MCP2515T-I/SO, U3 MX128-5.08-10P-GN01-CU-Y-A, U4 SN65HVD230DR, X1 X322516MLB4SI

Commit message: add copper pour (forgot in last commit) and tranfer via for signal
Parts:
- removed U3: MX128-5.08-10P-GN01-CU-Y-A, symbol ImportSymbol:MX128-5.08-10P-GN01-CU-Y-A
Changed lines of the file:
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@@
-	)
-	(symbol
-		(lib_id "ImportSymbol:MX128-5.08-10P-GN01-CU-Y-A")
-		(at 233.68 97.79 0)
-		(unit 1)
-		(exclude_from_sim no)
-		(in_bom yes)
-		(on_board yes)
-		(dnp no)
-		(fields_autoplaced yes)
-		(property "Reference" "U3"
-			(at 237.49 96.5199 0)
-			(effects
-				(font
-					(size 1.27 1.27)
-				)
-				(justify left)
-			)
-		)
-		(property "Value" "MX128-5.08-10P-GN01-CU-Y-A"
-			(at 237.49 99.0599 0)
-			(effects
-				(font
-					(size 1.27 1.27)
-				)
-				(justify left)
-			)
-		)
-		(property "Footprint" ""
-			(at 233.68 97.79 0)
-			(effects
-				(font
-					(size 1.27 1.27)
-				)
-				(hide yes)
-			)
-		)
-		(property "Datasheet" ""
-			(at 233.68 97.79 0)
-			(effects
-				(font
-					(size 1.27 1.27)
-				)
-				(hide yes)
-			)
-		)
-		(property "Description" ""
-			(at 233.68 97.79 0)
-			(effects
-				(font
-					(size 1.27 1.27)
-				)
-				(hide yes)
-			)
-		)
-		(property "Manufacturer Part" "MX128-5.08-10P-GN01-Cu-Y-A"
-			(at 233.68 97.79 0)
-			(effects
-				(font
-					(size 1.27 1.27)
-				)
-				(hide yes)
-			)
-		)
-		(property "Manufacturer" "MAX(迈旭)"
-			(at 233.68 97.79 0)
-			(effects
-				(font
-					(size 1.27 1.27)
-				)
-				(hide yes)
-			)
-		)
-		(property "Supplier Part" "C5290383"
-			(at 233.68 97.79 0)
-			(effects
-				(font
-					(size 1.27 1.27)
-				)
-				(hide yes)
-			)
-		)
-		(property "Supplier" "LCSC"
-			(at 233.68 97.79 0)
-			(effects
-				(font
-					(size 1.27 1.27)
-				)
-				(hide yes)
-			)
-		)
-		(pin "3"
-		)
-		(pin "10"
-		)
-		(pin "6"
-		)
-		(pin "1"
-		)
-		(pin "2"
-		)
-		(pin "9"
-		)
-		(pin "5"
-		)
-		(pin "4"
-		)
-		(pin "7"
-		)
-		(pin "8"
-		)
-		(instances
-			(project ""
-				(path "/e63e39d7-6ac0-4ffd-8aa3-1841a4541b55"
-					(reference "U3")
-					(unit 1)
-				)
-			)
-		)
 	)
 	(symbol
