File: _autosave-CAN_Shield.kicad_pcb (KiCad board)
At the start: 2 copper layers, 65 x 56.5 mm, 22 parts, among them J1 GPIO, J2 KF128-2.54-4P, U1 MX128-5.08-09P-GN01-CU-Y-A, U2 MCP2515T-I/SO, U4 SN65HVD230DR, X1 X322516MLB4SI

Commit message: quickly add 4 pin screw terminal block for I2C and move old SDA and SCL to new screw terminal block
Parts:
- moved J2 7.42 mm to (104.0, 64.3), turned to -90 degrees
Connections:
- J2 pad 1: unconnected-(J2-Pad1) -> +3V3
- J2 pad 2: unconnected-(J2-Pad2) -> /GPIO2/SDA1
- J2 pad 3: unconnected-(J2-Pad3) -> GND
- J2 pad 4: unconnected-(J2-Pad4) -> /GPIO3/SCL1
- U1 pad 1: /GPIO2/SDA1 -> /GPIO4/GPCLK0
- U1 pad 2: /GPIO3/SCL1 -> unconnected-(U1-Pad2)
Routing:
- net /GPIO2/SDA1: track 49.7 -> 17.1 mm
- net /GPIO3/SCL1: track 50.0 -> 23.3 mm
- net +3V3: track 50.0 -> 64.2 mm
Other:
- board text added: "3V3"
