File: CAN_Shield.kicad_sch (KiCad schematic)
At the start: 22 parts, among them J1 GPIO, U1 ATECC608A-SSHDA-T, U2 MCP2515T-I/SO, U4 SN65HVD230DR, X1 X322516MLB4SI, j2 DB128V-5.08-5P-GN-S, j3 DB128V-5.08-7P-GN-S, j4 DB128V-5.08-7P-GN-S

Commit message: add both bulk and bypass cap for sn65, increase spaing for crystal and add guard trace for crystal
Parts:
- removed C3: 100nF, PCM_JLCPCB:C_0603, symbol PCM_JLCPCB-Capacitors:0603,100nF
- added C3: 10nF, PCM_JLCPCB:C_0402, symbol PCM_JLCPCB-Capacitors:0402,10nF
- added C5: 100nF, PCM_JLCPCB:C_0402, symbol PCM_JLCPCB-Capacitors:0402,100nF
Connections:
- net +3V3: now also C3.1, C5.1
- net GND: now also C3.2, C5.2
